File: PCB/aprs_tracker_v3/aprs_tracker_v3.brd (EAGLE design)
At the start: 103.8 x 36.3 mm, 34 parts, among them IC1 7805T, T1 2N2222, X1 BU-SMA-V

Commit message: added finalized v3
Parts:
- C4: device rcl:C1206 -> rcl:0207/7
- R8: device rcl:0207/12 -> rcl:0207/7
- moved LED3 26.3 mm to (33.1, 26.8), flipped to the top
- moved R14 25.8 mm to (30.9, 26.9), flipped to the top, turned to 90 degrees
- moved R15 23.4 mm to (38.4, 2.03), turned to 180 degrees
- moved LED4 20.6 mm to (33.0, 4.06), turned to 180 degrees
- moved R8 17.3 mm to (40.1, 27.3)
- moved HC-06(BLUETOOTH) 16.1 mm to (39.1, 31.6), turned to 0 degrees
- moved C5 14.9 mm to (17.7, 29.8), turned to 180 degrees
- moved C7 14.2 mm to (25.7, 29.6), turned to 270 degrees
- moved LED2 12.5 mm to (30.5, 4.06), turned to 180 degrees
- moved C4 3.83 mm to (58.7, 28.1), turned to 0 degrees
- moved R1 3.30 mm to (19.1, 16.4)
- moved R2 3.06 mm to (8.13, 16.0)
- moved PWR_IN 2.79 mm to (56.4, 31.4), turned to 180 degrees
- moved C6 2.47 mm to (73.7, 31.4)
- moved R13 1.81 mm to (22.0, 2.16), turned to 0 degrees
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Routing:
- net VCC: track 204.6 -> 147.8 mm, vias 0 -> 1
- net N$26: track 106.9 -> 52.1 mm, vias 2 -> 0
- net GPS_TX: track 129.6 -> 81.7 mm, vias 1 -> 0
- net RADIO_SQL: track 51.1 -> 98.8 mm
- net N$13: track 46.5 -> 9.96 mm
- net N$3: track 38.2 -> 9.91 mm
- net MU_RX_1: track 35.8 -> 57.8 mm
- net MC_APRS_OUT: track 34.9 -> 16.4 mm
- net N$25: track 17.5 -> 2.51 mm
- net N$2: track 39.8 -> 54.1 mm, vias 0 -> 2
- net MU_TX_1: track 46.4 -> 60.2 mm
- net N$10: track 116.7 -> 105.3 mm
- net N$19: track 57.6 -> 69.0 mm
- net N$11: track 26.4 -> 33.2 mm
- net RADIO_PTT: track 23.5 -> 17.4 mm
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Other:
- board size 103.8 x 36.3 mm -> 103.8 x 35.7 mm
