File: PCB/aprs_tracker_v3/aprs_tracker_v3.brd (EAGLE design)
At the start: 103.8 x 35.7 mm, 34 parts, among them IC1 7805T, T1 2N2222, X1 BU-SMA-V

Commit message: added BOM and final fixes
Parts:
- C4: device rcl:0207/7 -> rcl:C1206
- C5, C7: value (none) -> 10u
- moved C4 9.44 mm to (66.3, 33.7)
- moved PWR_IN 1.00 mm to (57.4, 31.4)
- moved R9 0.80 mm to (49.0, 29.5)
Routing:
- net N$11: track 33.2 -> 26.2 mm
- net N$10: track 105.3 -> 108.0 mm
- net N$2: track 54.1 -> 54.3 mm, vias 2 -> 3
Other:
- board text added: "APRS v3.0"
- board text added: "KE8TJE"
