File: PCB/aprs_tracker_v4/aprs_tracker_v4.sch (EAGLE design)
At the start: 43 parts, among them IC1 7805T, IC2 ATMEGA328PB-AUR, IC3 74LVCH1T45GW,125, IC4 REG1117, T1 2N2222, X1 BU-SMA-V, Y1 ATS080B-E

Commit message: completed aprs v4
Parts:
- removed C3: 4.7u, rcl:C-US050-024X044
- removed JP2: (no value), pinhead:PINHD-2X3/90
- added JP4: (no value), pinhead:PINHD-2X3/90
- added JP5: (no value), pinhead:PINHD-2X4
- C4: device rcl:C-USC1206 -> rcl:C-USC0805
- C5, C7, C8, C9: device rcl:CPOL-EUE5-6 -> rcl:C-USC0805
- C6: device rcl:C-US050-024X044 -> rcl:C-USC0805
- JP1: device pinhead:PINHD-2X2 -> pinhead:PINHD-2X3/90
- R1, R10, R11, R3, R5, R7, R8: device rcl:R-EU_0207/7 -> rcl:R-US_R0805
- R12, R13, R14, R15, R2, R6: device rcl:R-EU_R0805 -> rcl:R-US_R0805
- R4: device rcl:R-EU_0204/7 -> rcl:R-US_R0805
- renumbered LED1 to D3, LED2 to D2, LED3 to D4, LED4 to D1, LED5 to D5
Connections:
- new net A63: D2.A, U1.3D-FIX
- net +3V3: now also C9.1; no longer C9.+
- net A6: no longer D2.A, U1.3D-FIX
- net GND: now also C5.2, C7.2, C8.2, C9.2, JP1.5, JP4.5, JP4.6, JP5.1; no longer C5.-, C7.-, C8.-, C9.-, JP1.1, JP1.3, JP2.1
- net N$10: no longer C3.2
- net N$11: no longer C3.1, R9.A
- net PIN11: now also JP4.3, JP5.3; no longer JP1.4, JP2.3
- net PIN12: now also JP4.4, JP5.6; no longer JP1.2, JP2.6
- net PIN9: now also JP1.4
- net RESET: now also JP5.2; no longer JP2.2
- net RX: now also JP5.7
- net SCK: now also JP5.4; no longer JP2.4
- net SCL: now also JP1.1
- net SDA: now also JP1.2
- net TX: now also JP5.8
- net VCC: now also C7.1, C8.1, JP1.6, JP5.5; no longer C7.+, C8.+, JP2.5
- net V_BAT: now also C5.1, JP1.3; no longer C5.+
