File: PCB/aprs_tracker_v5/aprs_tracker_v5.brd (EAGLE design)
At the start: 100 x 35 mm, 42 parts, among them IC2 ATMEGA328PB-AUR, IC4 REG1117, T1 2N2222, Y1 ATS080B-E

Commit message: added 10k res to the i2c lines
Parts:
- added R13, R16: 10k, rcl:R0805
Connections:
- net +3V3: now also R13.2, R16.2
- net SCL: now also R16.1
- net SDA: now also R13.1
Routing:
- net +3V3: track 100.6 -> 105.7 mm
- net SDA: track 10.5 -> 13.5 mm
- net SCL: track 11.4 -> 12.2 mm
Changed lines of the file:
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@@
 <attribute name="VALUE" x="39.878" y="30.226" size="1.27" layer="28" rot="MR180"/>
+</element>
+<element name="R13" library="rcl" library_urn="urn:adsk.eagle:library:334" package="R0805" package3d_urn="urn:adsk.eagle:package:23553/2" value="10k" x="10.922" y="22.606" smashed="yes" rot="MR270">
+<attribute name="NAME" x="9.652" y="23.241" size="1.27" layer="26" rot="MR270"/>
+<attribute name="POPULARITY" value="85" x="10.922" y="22.606" size="1.778" layer="28" rot="MR270" display="off"/>
+<attribute name="SPICEPREFIX" value="R" x="10.922" y="22.606" size="1.778" layer="28" rot="MR270" display="off"/>
+<attribute name="VALUE" x="13.462" y="23.241" size="1.27" layer="28" rot="MR270"/>
+</element>
+<element name="R16" library="rcl" library_urn="urn:adsk.eagle:library:334" package="R0805" package3d_urn="urn:adsk.eagle:package:23553/2" value="10k" x="11.43" y="18.542" smashed="yes" rot="R270">
+<attribute name="NAME" x="12.7" y="19.177" size="1.27" layer="25" rot="R270"/>
+<attribute name="POPULARITY" value="85" x="11.43" y="18.542" size="1.778" layer="27" rot="R270" display="off"/>
+<attribute name="SPICEPREFIX" value="R" x="11.43" y="18.542" size="1.778" layer="27" rot="R270" display="off"/>
+<attribute name="VALUE" x="8.89" y="19.177" size="1.27" layer="27" rot="R270"/>
 </element>
 </elements>
@@
 <vertex x="-1.524" y="-2.286"/>
 </polygon>
-<via x="12.192" y="17.526" extent="1-16" drill="0.35"/>
+<via x="12.7" y="19.558" extent="1-16" drill="0.35"/>
 <via x="14.732" y="21.844" extent="1-16" drill="0.35"/>
 </signal>
@@
 <contactref element="JP3" pad="3"/>
 <wire x1="18.4785" y1="14.478" x2="18.4785" y2="13.335" width="0.2286" layer="16"/>
-<wire x1="14.19225" y1="18.76425" x2="18.4785" y2="14.478" width="0.2286" layer="1"/>
-<wire x1="9.23925" y1="18.76425" x2="14.19225" y2="18.76425" width="0.2286" layer="1"/>
-<wire x1="8.9535" y1="19.05" x2="9.23925" y2="18.76425" width="0.2286" layer="1"/>
-<wire x1="8.66775" y1="18.76425" x2="8.9535" y2="19.05" width="0.2286" layer="1"/>
-<wire x1="7.8105" y1="18.76425" x2="8.66775" y2="18.76425" width="0.2286" layer="1"/>
+<wire x1="14.44625" y1="18.51025" x2="18.4785" y2="14.478" width="0.2286" layer="1"/>
+<wire x1="9.49325" y1="18.51025" x2="14.44625" y2="18.51025" width="0.2286" layer="1"/>
+<wire x1="9.23925" y1="18.76425" x2="9.49325" y2="18.51025" width="0.2286" layer="1"/>
+<wire x1="7.8105" y1="18.76425" x2="9.23925" y2="18.76425" width="0.2286" layer="1"/>
 <wire x1="7.52475" y1="19.05" x2="7.8105" y2="18.76425" width="0.2286" layer="1"/>
 <wire x1="7.239" y1="19.05" x2="7.52475" y2="19.05" width="0.2286" layer="1"/>
@@
 <wire x1="18.4785" y1="21.05025" x2="18.4785" y2="21.717" width="0.2286" layer="16"/>
 <wire x1="18.0975" y1="20.66925" x2="18.4785" y2="21.05025" width="0.2286" layer="16"/>
-<wire x1="17.145" y1="20.66925" x2="18.0975" y2="20.66925" width="0.2286" layer="1"/>
-<wire x1="16.5735" y1="20.09775" x2="17.145" y2="20.66925" width="0.2286" layer="1"/>
-<wire x1="8.28675" y1="20.09775" x2="16.5735" y2="20.09775" width="0.2286" layer="1"/>
 <wire x1="18.4785" y1="21.717" x2="18.54" y2="21.808" width="0.2286" layer="16"/>
 <wire x1="8.28675" y1="20.09775" x2="8.27" y2="20.04" width="0.2286" layer="1"/>
 <via x="18.0975" y="20.66925" extent="1-16" drill="0.3"/>
+<contactref element="R16" pad="1"/>
+<wire x1="8.27" y1="20.04" x2="9.424" y2="20.04" width="0.2286" layer="1"/>
+<wire x1="9.972" y1="19.492" x2="11.43" y2="19.492" width="0.2286" layer="1"/>
+<wire x1="9.424" y1="20.04" x2="9.972" y2="19.492" width="0.2286" layer="1"/>
+<wire x1="11.43" y1="19.492" x2="12.512" y2="20.574" width="0.2286" layer="1"/>
+<wire x1="15.78118125" y1="20.574" x2="16.17883125" y2="20.17635" width="0.2286" layer="1"/>
+<wire x1="12.512" y1="20.574" x2="15.78118125" y2="20.574" width="0.2286" layer="1"/>
+<wire x1="17.6046" y1="20.17635" x2="18.0975" y2="20.66925" width="0.2286" layer="1"/>
+<wire x1="16.17883125" y1="20.17635" x2="17.6046" y2="20.17635" width="0.2286" layer="1"/>
 </signal>
 <signal name="SDA">
@@
 <wire x1="8.28675" y1="22.57425" x2="8.27" y2="22.58" width="0.2286" layer="1"/>
 <via x="17.24025" y="22.95525" extent="1-16" drill="0.3"/>
+<contactref element="R13" pad="1"/>
+<wire x1="10.922" y1="23.556" x2="9.246" y2="23.556" width="0.254" layer="16"/>
+<wire x1="9.246" y1="23.556" x2="8.27" y2="22.58" width="0.254" layer="16"/>
 </signal>
 <signal name="SCK">
@@
 <wire x1="8.28675" y1="17.43075" x2="8.27" y2="17.5" width="0.508" layer="16"/>
 <wire x1="15.33525" y1="23.8125" x2="15.33525" y2="24.86025" width="0.508" layer="16"/>
-<wire x1="10.19175" y1="18.669" x2="15.33525" y2="23.8125" width="0.508" layer="16"/>
+<wire x1="10.19175" y1="18.669" x2="12.652375" y2="21.129625" width="0.508" layer="16"/>
+<wire x1="12.652375" y1="21.129625" x2="15.33525" y2="23.8125" width="0.508" layer="16"/>
 <wire x1="9.525" y1="18.669" x2="10.19175" y2="18.669" width="0.508" layer="16"/>
 <wire x1="8.47725" y1="17.62125" x2="9.525" y2="18.669" width="0.508" layer="16"/>
@@
 <wire x1="23.4315" y1="16.28775" x2="23.19" y2="16.358" width="0.508" layer="16"/>
 <via x="51.2445" y="19.71675" extent="1-16" drill="0.3"/>
+<contactref element="R13" pad="2"/>
+<contactref element="R16" pad="2"/>
+<wire x1="8.27" y1="17.5" x2="11.338" y2="17.5" width="0.508" layer="1"/>
+<wire x1="11.338" y1="17.5" x2="11.43" y2="17.592" width="0.508" layer="1"/>
+<wire x1="10.922" y1="21.656" x2="12.126" y2="21.656" width="0.508" layer="16"/>
+<wire x1="12.126" y1="21.656" x2="12.652375" y2="21.129625" width="0.508" layer="16"/>
 </signal>
 <signal name="N$6">

Commit message: added v5 final production PCB
Parts:
- removed D1: (no value), led:CHIP-LED0805
- removed R15: 1k, rcl:R0805
- added D2: (no value), led:CHIP-LED0805
- added IC3: 74LVCH1T45GW,125, 74LVCH1T45GW_125:74LVCH1T45GW125
- added R17: 1k, rcl:R0805
- PWR_IN: value (none) -> PINHD-1X2; device pinhead:1X02 -> Connector:1X02
- X1: value (none) -> BU-SMA-V; device pinhead:1X02 -> con-coax:BU-SMA-V
- moved X1 5.64 mm to (90.4, 8.13), turned to 0 degrees
- moved R12 5.14 mm to (65.3, 27.6)
- moved PWR_IN 5.13 mm to (12.4, 30.2), turned to 0 degrees
- moved T1 3.94 mm to (23.4, 31.8)
- moved R10 2.81 mm to (23.4, 25.7), turned to 90 degrees
- moved R11 2.74 mm to (26.2, 25.9)
- moved R6 2.52 mm to (16.8, 25.7), turned to 0 degrees
- moved C9 1.39 mm to (53.4, 19.8), turned to 0 degrees
- moved R16 1.37 mm to (12.7, 19.1)
- moved R13 1.27 mm to (11.7, 23.6), turned to 90 degrees
- moved D3 1.14 mm to (69.5, 27.6), turned to 90 degrees
- moved R8 0.76 mm to (50.4, 31.5)
- moved C4 0.25 mm to (41.4, 27.7)
- moved C8 0.12 mm to (49.0, 19.8), turned to 180 degrees
Connections:
- removed net AUDIO_IN: JP3.1
- removed net N$3: D1.C, R15.2
- new net N$1: IC3.4, U1.P$9
- new net N$9: D2.C, R17.2
- net +3V3: now also IC3.6; no longer D1.A, IC2.18, IC2.4, IC2.6, JP1.5, JP3.6, R13.2, R16.2, R6.2
- net GND: now also IC3.2, IC3.5, X1.3, X1.4, X1.5
- net GPS_RX: now also IC3.3, R17.1; no longer R15.1, U1.P$9
- net MC_APRS_OUT: now also JP3.1
- net VCC: now also D2.A, IC2.18, IC2.4, IC2.6, IC3.1, JP1.5, JP3.6, R13.2, R16.2, R6.2
Routing:
- net +3V3: track 105.7 -> 28.4 mm, vias 1 -> 0
- net VCC: track 119.0 -> 168.7 mm, vias 2 -> 1
- net MC_APRS_OUT: track 21.8 -> 59.7 mm
- net N$10: track 33.5 -> 25.5 mm
- net RX: track 29.5 -> 22.7 mm, vias 1 -> 2
- net N$8: track 15.4 -> 10.6 mm
- net GPS_TX: track 61.8 -> 57.2 mm
- net MU_TX_1: track 53.7 -> 49.2 mm
- net N$1: track 0.00 -> 4.50 mm
- net GPS_RX: track 57.2 -> 61.6 mm, vias 1 -> 5
- net RADIO_WAKE: track 77.3 -> 73.0 mm
- net RADIO_OUTPUT_POWER: track 73.9 -> 78.1 mm
- net RESET: track 40.0 -> 36.2 mm, vias 1 -> 2
- net MU_RX_1: track 46.9 -> 43.3 mm
- net N$3: track 2.52 -> 0.00 mm
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Other:
- board text added: "APRS tracker v5.0 KE8TJE - Jan 2025"
- board text added: "Vcc"
- board text removed: "3.3V"
- board text removed: "APRS tracker v5.0 KE8TJE - Dec 2024"
- board text removed: "P1"
- board text removed: "P2"
- board text removed: "RX"
- board text removed: "V_Bat"
